File: pcb/EFM32TG11-Core-MCU.kicad_sch (KiCad schematic)
At the start: 26 parts, among them J5 BOOT, J6 Conn_ARM_JTAG_SWD_10, SW1 SW_Push, U2 EFM32TG11B340F64GQ64, Y1 32.7680KHz, Y2 48MHz

Commit message: Fix Nets for Hierarchical Sheets
Defined busses to pass nets to and from MCU sheet and IO connector
sheet.
Connections:
- net PA12: no longer names the net of U2.17 (PA12)
- net PA13: no longer names the net of U2.18 (PA13(5V))
- net PA14: no longer names the net of U2.19 (PA14)
- net PE14: no longer names the net of U2.63 (PE14)
- net PF4: no longer names the net of U2.53 (PF4)
- no-connect marks 0 -> 5
Other:
- moved on the sheet: NT1
